File: PCB/lighthouse_board/Lighthouse.brd (EAGLE design)
At the start: 53.3 x 70.5 mm, 15 parts, among them U1 A4988_STEPPER_MOTOR_DRIVER_CA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

Commit message: new version of stepper pcb and lighthouse pcb
Changed lines of the file:
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@@
 <dimension x1="53.34" y1="70.485" x2="0" y2="70.485" x3="26.67" y3="81.28" textsize="1.27" textratio="9" layer="47"/>
 <dimension x1="50.8" y1="3.175" x2="53.34" y2="3.175" x3="52.07" y3="-10.795" textsize="1.27" textratio="9" layer="47"/>
+<text x="48.26" y="44.45" size="1.27" layer="25">+5V</text>
+<text x="48.26" y="59.055" size="1.27" layer="25">GND</text>
 </plain>
 <attributes>

Commit message: update pcb for order
Parts:
- removed J2: (no value), SparkFun-Connectors:1X02_6.35_SCREWTERM
- removed J6: (no value), SparkFun-Connectors:JST-4-PTH-VERT
- added J5, J7: (no value), SparkFun-Connectors:SCREWTERMINAL-5MM-2
- J1: value (none) -> B4B-XH-A(LF)(SN); device SparkFun-Connectors:1X02_6.35_SCREWTERM -> B4B-XH-A_LF__SN_:JST_B4B-XH-A(LF)(SN)
- moved J1 38.1 mm to (29.2, 66.7), turned to 180 degrees
- moved J3 8.28 mm to (49.5, 47.6), turned to 90 degrees
- moved J4 7.65 mm to (44.5, 66.7), turned to 180 degrees
- moved +5V 2.29 mm to (41.3, 53.3)
- moved R3 2.01 mm to (41.3, 44.5)
- moved R1 1.91 mm to (25.4, 36.2)
- moved R5 1.91 mm to (20.3, 27.9)
- moved U1 1.91 mm to (25.4, 50.2)
- moved R4 1.90 mm to (23.5, 31.8)
- moved C1 0.63 mm to (13.3, 64.1)
- moved R2 0.63 mm to (6.35, 45.1)
- moved VMOT 0.63 mm to (6.35, 54.6)
Connections:
- net 12V: now also J7.2; no longer J2.P2
- net 5V: now also J5.2; no longer J1.P2
- net GND: now also J5.1, J7.1; no longer J1.P1, J2.P1
- net N$10: now also J1.2; no longer J6.3
- net N$7: now also J1.4; no longer J6.1
- net N$8: now also J1.3; no longer J6.2
- net N$9: now also J1.1; no longer J6.4
Routing:
- net 12V: track 40.3 -> 52.5 mm
- net 5V: track 22.5 -> 18.4 mm
- net LEDS: track 36.0 -> 34.3 mm
- net N$9: track 11.2 -> 10.2 mm
- net N$7: track 11.2 -> 10.2 mm
- net HALL: track 48.2 -> 47.4 mm
- net N$10: track 11.0 -> 10.2 mm
- net N$8: track 11.0 -> 10.2 mm
- net STEP: track 24.1 -> 23.3 mm
- net SLEEP: track 27.2 -> 26.4 mm
- net DIR: track 23.6 -> 22.8 mm
- net N$1: track 5.38 -> 4.74 mm
- added copper zone on layer 16, net 5V
- added copper zone on layer 1, net GND
Other:
- board text added: "Lighthouse Board - V3 BOTSEIDON"
- board text removed: "Lighthouse Board - V2.1 BOTSEIDON"
