File: PCB/stepper_motor_board/Stepper_motor.brd (EAGLE design)
At the start: 59.7 x 103.8 mm, 27 parts, among them U1 A4988_STEPPER_MOTOR_DRIVER_CA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, U2 A4988_STEPPER_MOTOR_DRIVER_CA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, U3 A4988_STEPPER_MOTOR_DRIVER_CA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

Commit message: new version of stepper pcb and lighthouse pcb
Parts:
- removed C2, C3: 100uF, SparkFun-Capacitors:PANASONIC_D
- removed J1, J8: (no value), SparkFun-Connectors:JST-4-PTH-VERT
- removed J3, J6: (no value), SparkFun-Connectors:SCREWTERMINAL-3.5MM-3
- removed R4, R5, R6, R7, R8, R9: 0, SparkFun-Resistors:1206
- removed U2, U3: A4988_STEPPER_MOTOR_DRIVER_CARRIER, A4988_STEPPER_MOTOR_DRIVER_CARRIER:MODULE_A4988_STEPPER_MOTOR_DRIVER_CARRIER
- moved J4 1.27 mm to (3.81, 66.0)
- moved +5V 1.27 mm to (7.62, 90.2)
- moved R10 1.27 mm to (7.62, 94.0)
- moved R11 1.27 mm to (52.1, 94.0)
- moved VMOT 1.27 mm to (52.1, 90.2)
Connections:
- removed net N$15: J3.2, U2.7
- removed net N$16: J3.1, U2.8
- removed net N$17: J3.3, U2.5, U2.6
- removed net N$18: R6.1, U2.2
- removed net N$19: R5.1, U2.3
- removed net N$20: R4.1, U2.4
- removed net N$25: J6.2, U3.7
- removed net N$26: J6.1, U3.8
- removed net N$27: J6.3, U3.5, U3.6
- removed net N$28: R9.1, U3.2
- removed net N$29: R8.1, U3.3
- removed net N$30: R7.1, U3.4
- removed net N$31: J8.4, U3.11
- removed net N$32: J8.3, U3.12
- removed net N$33: J8.2, U3.13
- removed net N$34: J8.1, U3.14
- removed net N$35: J1.4, U2.11
- removed net N$36: J1.3, U2.12
- removed net N$37: J1.2, U2.13
- removed net N$38: J1.1, U2.14
- net 12V: no longer C2.+, C3.+, U2.16, U3.16
- net 5V: no longer R4.2, R5.2, R6.2, R7.2, R8.2, R9.2, U2.10, U3.10
- net GND: no longer C2.-, C3.-, U2.15, U2.9, U3.15, U3.9
Routing:
- net 12V: track 113.4 -> 38.4 mm, vias 3 -> 0
- net N$27: track 21.8 -> 0.00 mm
- net N$17: track 21.8 -> 0.00 mm
- net N$35: track 21.4 -> 0.00 mm
- net N$38: track 21.4 -> 0.00 mm
- net N$34: track 21.4 -> 0.00 mm
- net N$31: track 21.4 -> 0.00 mm
- net N$36: track 21.2 -> 0.00 mm
- net N$33: track 21.2 -> 0.00 mm
- net N$32: track 21.2 -> 0.00 mm
- net N$37: track 21.2 -> 0.00 mm
- net N$15: track 19.4 -> 0.00 mm
- net N$25: track 19.4 -> 0.00 mm
- net N$30: track 19.1 -> 0.00 mm
- net N$26: track 19.1 -> 0.00 mm
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- removed copper zone on layer 1, net 5V
- removed copper zone on layer 16, net GND
Other:
- board size 59.7 x 103.8 mm -> 59.7 x 47.9 mm
- board text added: "Stepper Motor Board - V1.3 BOTSEIDON"
- board text removed: "Stepper Motor Board - V1.2 BOTSEIDON"

Commit message: update pcb for order
Parts:
- removed J5: (no value), SparkFun-Connectors:JST-4-PTH-VERT
- removed J7: (no value), SparkFun-Connectors:1X02_6.35_SCREWTERM
- added J1: (no value), SparkFun-Connectors:SCREWTERMINAL-5MM-2
- added J3: B4B-XH-A(LF)(SN), B4B-XH-A_LF__SN_:JST_B4B-XH-A(LF)(SN)
- J2: device SparkFun-Connectors:1X02_6.35_SCREWTERM -> SparkFun-Connectors:SCREWTERMINAL-5MM-2
- moved R10 12.0 mm to (19.1, 90.2)
- moved R11 11.5 mm to (40.6, 92.7)
- moved J4 6.35 mm to (3.81, 72.4), turned to 270 degrees
- moved VMOT 3.59 mm to (49.5, 92.7), turned to 90 degrees
- moved J2 2.54 mm to (36.8, 100.3), turned to 180 degrees
- moved +5V 1.27 mm to (8.89, 90.2), turned to 270 degrees
- moved C1 1.27 mm to (47.0, 83.8)
Connections:
- net 12V: now also J2.2; no longer J2.P2
- net 5V: now also J1.2; no longer J7.P2
- net GND: now also J1.1, J2.1; no longer J2.P1, J7.P1
- net N$1: now also J3.1; no longer J5.4
- net N$2: now also J3.2; no longer J5.3
- net N$3: now also J3.3; no longer J5.2
- net N$4: now also J3.4; no longer J5.1
- net N$6: now also J4.3; no longer J4.1
- net N$7: now also J4.1; no longer J4.3
Routing:
- net 5V: track 0.00 -> 17.4 mm, vias 0 -> 3
- net 12V: track 38.4 -> 34.9 mm
- net N$11: track 4.37 -> 6.01 mm
- net N$1: track 21.4 -> 20.3 mm
- net N$4: track 21.4 -> 20.4 mm
- net N$2: track 21.2 -> 20.3 mm
- net N$3: track 21.2 -> 20.4 mm
- added copper zone on layer 16, net 5V
- added copper zone on layer 1, net GND
Other:
- board text added: "DIR"
- board text added: "NSLEEP"
- board text added: "STEP"
- board text added: "Stepper Motor Board - V3 BOTSEIDON"
- board text removed: "Stepper Motor Board - V1.3 BOTSEIDON"
